File: CONTROL_ESP32.kicad_sch (KiCad schematic)
At the start: 28 parts, among them J1 Screw_Terminal_01x02, J2 Screw_Terminal_01x04, J3 Screw_Terminal_01x04, SW1 SW_Push_SPDT, SW2 SW_Push, SW3 SW_Push, SW4 SW_Push, SW5 SW_Push, U1 ESP32-DEVKITC-32D, U2 LM7805_TO220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

Commit message: Un pequeño Cambio
Parts:
- R10, R9: value (none) -> COM-09806; footprint (none) -> COM-09806:TRIM_COM-09806
Changed lines of the file:
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@@
       (effects (font (size 1.27 1.27)) hide)
     )
-    (property "Value" "" (id 1) (at 85.09 134.62 0))
+    (property "Value" "+3.3V" (id 1) (at 85.09 134.62 0))
     (property "Footprint" "" (id 2) (at 85.09 139.7 0)
       (effects (font (size 1.27 1.27)) hide)
@@
     (in_bom yes) (on_board yes) (fields_autoplaced)
     (property "Reference" "R10" (id 0) (at 105.41 163.83 0))
-    (property "Value" "" (id 1) (at 105.41 166.37 0))
-    (property "Footprint" "" (id 2) (at 105.41 170.18 0)
+    (property "Value" "COM-09806" (id 1) (at 105.41 166.37 0))
+    (property "Footprint" "COM-09806:TRIM_COM-09806" (id 2) (at 105.41 170.18 0)
       (effects (font (size 1.27 1.27)) (justify left bottom) hide)
     )
@@
     (in_bom yes) (on_board yes) (fields_autoplaced)
     (property "Reference" "R9" (id 0) (at 105.41 137.16 0))
-    (property "Value" "" (id 1) (at 105.41 139.7 0))
-    (property "Footprint" "" (id 2) (at 105.41 143.51 0)
-      (effects (font (size 1.27 1.27)) (justify left bottom) hide)
-    )
+    (property "Value" "COM-09806" (id 1) (at 105.41 139.7 0))
+    (property "Footprint" "COM-09806:TRIM_COM-09806" (id 2) (at 105.41 143.51 0)
+      (effects (font (size 1.27 1.27)) (justify left bottom) hide)
+    )

Commit message: add copia
Connections:
- net +5V: now also C3.1, R1.1, U2.3 (VO)
- net VCC: now reaches J1.2 (Pin_2), SW1.2 (B)
- net VEE: now reaches C2.1, D1.1 (K), U2.1 (VI)
Other:
- moved on the sheet: C2
